Commit message: Almost complete

File: urdf/robot.urdf (robot description, URDF)
Before this commit: robot my_robot, 8 links, 7 joints
Links:
- removed link laser_horiz
- added link label_horiz, mass 0.01; visual mesh filename=package://velodyne_description/meshes/VLP16_scan.dae
- added link label_horiz_base_link, mass 0.83; collision cylinder length=0.0717 radius=0.0516; visual mesh filename=package://velodyne_description/meshes/VLP16_base_1.dae
- link base: geometry collision box size=0.94 0.78 1.98; visual box size=0.10 0.78 1.9
- link laser_vert_bottom: mass None -> 1e-5; geometry collision box size=0.1 0.1 0.1; visual mesh filename=package://gazebo_plugins/test/multi_robot_scenario/meshes/l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
- link laser_vert_top_left: mass None -> 1e-5; geometry collision box size=0.1 0.1 0.1; visual mesh filename=package://gazebo_plugins/test/multi_robot_scenario/meshes/l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
- link laser_vert_top_right: mass None -> 1e-5; geometry collision box size=0.1 0.1 0.1; visual mesh filename=package://gazebo_plugins/test/multi_robot_scenario/meshes/l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
- link wheel_center: geometry collision cylinder length=0.05 radius=0.15; visual cylinder length=0.05 radius=0.15
- link wheel_left: geometry collision cylinder length=0.05 radius=0.2; visual cylinder length=0.05 radius=0.2
- link wheel_right: geometry collision cylinder length=0.05 radius=0.2; visual cylinder length=0.05 radius=0.2
Joints:
- removed joint base_laser_horiz_joint
- added joint label_horiz_base_mount_joint: type fixed, parent base, child label_horiz_base_link, origin xyz=0.2325 0.0001 0.9301 rpy=-0.0012 0.1146 -0.0015
- added joint label_horiz_base_scan_joint: type fixed, parent label_horiz_base_link, child label_horiz, origin xyz=0 0 0.0377 rpy=0 0 0
- joint base_laser_vert_bottom_joint: axis (none) -> 0 0 1; origin (none) -> xyz=0.3158 -0.0021 -0.4800 rpy=3.1355 -1.3045 0.0025
- joint base_laser_vert_top_left_joint: axis (none) -> 0 0 1; origin (none) -> xyz=0.2997 0.1531 0.8543 rpy=1.1780 0.6198 1.9560
- joint base_laser_vert_top_right_joint: axis (none) -> 0 0 1; origin (none) -> xyz=0.2978 -0.1450 0.8551 rpy=-1.1760 0.6313 -1.9377
- joint base_wheel_center_joint: axis (none) -> 0.0 0.0 1.0; origin (none) -> xyz=0.57 0.0 -0.99 rpy=-1.57 0.0 0.0; type fixed -> continuous
- joint base_wheel_left_joint: axis (none) -> 0.0 0.0 1.0; origin (none) -> xyz=-0.37 0.4 -0.99 rpy=-1.57 0.0 0.0; type fixed -> continuous
- joint base_wheel_right_joint: axis (none) -> 0.0 0.0 1.0; origin (none) -> xyz=-0.37 -0.4 -0.99 rpy=-1.57 0.0 0.0; type fixed -> continuous

File: urdf/robot.xacro (robot description, xacro)
@@ -1,89 +1,73 @@
 <?xml version="1.0"?>
 <robot xmlns:xacro="http://www.ros.org/wiki/xacro" name="my_robot">
-    <xacro:macro name="laser" params="label x y z r p yaw">
-        <link name="laser_${label}">
-            <origin xyz="${x} ${y} ${z}" rpy="${r} ${p} ${y}" />
+    <xacro:include filename="$(find gazebo_plugins)/test/multi_robot_scenario/xacro/laser/hokuyo.xacro" />
+    <xacro:include filename="$(find velodyne_description)/urdf/VLP-16.urdf.xacro" />
+    <xacro:macro name="reflect_wheel" params="suffix reflect">
+        <joint name="base_wheel_${suffix}_joint" type="continuous">
+            <origin xyz="-0.37 ${reflect*0.4} -0.99" rpy="-1.57 0.0 0.0" />
+            <axis xyz="0.0 0.0 1.0" />
+            <parent link="base" />
+            <child link="wheel_${suffix}" />
+        </joint>
+        <link name="wheel_${suffix}">
+            <origin xyz="-0.37 ${reflect*0.01} -0.99" rpy="0.0 0.0 0.0" />
             <visual>
                 <geometry>
-                    <cylinder radius="0.05" length="0.10" />
+                    <cylinder radius="0.2" length="0.05" />
                 </geometry>
             </visual>
             <collision>
                 <geometry>
-                    <cylinder radius="0.05" length="0.10" />
+                    <cylinder radius="0.2" length="0.05" />
                 </geometry>
             </collision>
         </link>
-        <joint name="base_laser_${label}_joint" type="fixed">
-            <parent link="base" />
-            <child link="laser_${label}" />
-        </joint>
     </xacro:macro>
     <link name="base">
+        <origin xyz="0.0 0.0 0.0" rpy="0.0 0.0 0.0" />
         <visual>
+            <origin xyz="0.0 0.0 -0.99" />
             <geometry>
-                <box size="0.05 0.05 0.05" />
+                <box size="0.94 0.78 0.25" />
+            </geometry>
+        </visual>
+        <visual>
+            <origin xyz="0.23 0.0 0.0" />
+            <geometry>
+                <box size="0.10 0.78 1.9"/>
             </geometry>
         </visual>
         <collision>
             <geometry>
-                <box size="0.05 0.05 0.05" />
+                <box size="0.94 0.78 1.98" />
             </geometry>
         </collision>
     </link>
-    <joint name="base_wheel_right_joint" type="fixed">
+    <xacro:reflect_wheel suffix="left" reflect="1" />
+    <joint name="base_wheel_center_joint" type="continuous">
+        <origin xyz="0.57 0.0 -0.99" rpy="-1.57 0.0 0.0" />
+        <axis xyz="0.0 0.0 1.0" />
         <parent link="base" />
-        <child link="wheel_right" />
+        <child link="wheel_center" />
     </joint>
-    <link name="wheel_right">
-        <origin xyz="-0.10 -0.4 0.0" rpy="-1.571 0.0 0.0" />
+    <link name="wheel_center">
+        <origin xyz="0.57 0.0 -0.99" rpy="0.0 0.0 0.0" />
         <visual>
             <geometry>
-                <sphere radius="0.05" />
+                <cylinder radius="0.15" length="0.05" />
             </geometry>
         </visual>
         <collision>
             <geometry>
-                <sphere radius="0.05" />
+                <cylinder radius="0.15" length="0.05" />
             </geometry>
         </collision>
     </link>
-    <joint name="base_wheel_left_joint" type="fixed">
-        <parent link="base" />
-        <child link="wheel_left" />
-    </joint>
-    <link name="wheel_left">
-        <origin xyz="-0.10 0.4 0.0" rpy="-1.571 0.0 0.0" />
-        <visual>
-            <geometry>
-                <sphere radius="0.05" />
-            </geometry>
-        </visual>
-        <collision>
-            <geometry>
-                <sphere radius="0.05" />
-            </geometry>
-        </collision>
-    </link>
-    <joint name="base_wheel_center_joint" type="fixed">
-        <parent link="base" />
-        <child link="wheel_center" />
-    </joint>
-    <link name="wheel_center">
-        <origin xyz="-0.10 0.0 0.0" rpy="-1.571 0.0 0.0" />
-        <visual>
-            <geometry>
-                <sphere radius="0.05" />
-            </geometry>
-        </visual>
-        <collision>
-            <geometry>
-                <sphere radius="0.05" />
-            </geometry>
-        </collision>
-    </link>
-    <xacro:laser label="horiz" x="0.2325" y="0.0001" z="1.9201" r="0.2325" p="-0.0001" yaw="1.9201" />
-    <xacro:laser label="vert_top_right" x="0.2978" y="-0.1450" z="1.8451" r="-1.1760" p="0.6313" yaw="-1.9377" />
-    <xacro:laser label="vert_top_left" x="0.2997" y="0.1531" z="1.8443" r="1.1780" p="0.6193" yaw="1.9560" />
-    <xacro:laser label="vert_bottom" x="0.3158" y="-0.0021" z="0.5100" r="3.1355" p="-1.3045" yaw="0.0025" />
+    <xacro:reflect_wheel suffix="right" reflect="-1" />
+    <xacro:VLP-16 parent="base" name="label_horiz" topic="laser_horiz/packets" hz="10" samples="440" gpu="false">
+        <origin xyz="0.2325 0.0001 0.9301" rpy="-0.0012 0.1146 -0.0015" />
+    </xacro:VLP-16>
+    <xacro:laser name="laser_vert_top_right" parent="base" xyz="0.2978 -0.1450 0.8551" rpy="-1.1760 0.6313 -1.9377" meshes="package://gazebo_plugins/test/multi_robot_scenario/meshes/laser" />
+    <xacro:laser name="laser_vert_top_left" parent="base" xyz="0.2997 0.1531 0.8543" rpy="1.1780 0.6198 1.9560" meshes="package://gazebo_plugins/test/multi_robot_scenario/meshes/laser" />
+    <xacro:laser name="laser_vert_bottom" parent="base" xyz="0.3158 -0.0021 -0.4800" rpy="3.1355 -1.3045 0.0025" meshes="package://gazebo_plugins/test/multi_robot_scenario/meshes/laser" />
 </robot>

Commit message: Updated dependencies and final layout

File: urdf/robot.urdf (robot description, URDF)
Before this commit: robot my_robot, 9 links, 8 joints
Joints:
- joint base_wheel_center_joint: origin xyz=0.57 0.0 -0.99 rpy=-1.57 0.0 0.0 -> xyz=0.57 0.0 -1.04 rpy=-1.57 0.0 0.0

File: urdf/robot.xacro (robot description, xacro)
@@ -46,5 +46,5 @@
     <xacro:reflect_wheel suffix="left" reflect="1" />
     <joint name="base_wheel_center_joint" type="continuous">
-        <origin xyz="0.57 0.0 -0.99" rpy="-1.57 0.0 0.0" />
+        <origin xyz="0.57 0.0 -1.04" rpy="-1.57 0.0 0.0" />
         <axis xyz="0.0 0.0 1.0" />
         <parent link="base" />
@@ -52,5 +52,5 @@
     </joint>
     <link name="wheel_center">
-        <origin xyz="0.57 0.0 -0.99" rpy="0.0 0.0 0.0" />
+        <origin xyz="0.57 0.0 -1.04" rpy="0.0 0.0 0.0" />
         <visual>
             <geometry>

Commit message: Through page 3 of lab

File: urdf/robot.urdf (robot description, URDF)
Before this commit: robot my_robot, 9 links, 8 joints
Links:
- added link base_link
- added link imu; collision sphere radius=0.1; visual sphere radius=0.1
Joints:
- added joint base_link_base_joint: type fixed, parent base_link, child base, origin xyz=0.07 0 1.792 rpy=0.0 3.14159265359 0.0
- added joint base_link_imu_joint: type fixed, parent base_link, child imu, origin xyz=0.0 0.0 0.0 rpy=3.1405788 0.0034281 3.1382064

File: urdf/robot.xacro (robot description, xacro)
@@ -1,73 +1,28 @@
 <?xml version="1.0"?>
-<robot xmlns:xacro="http://www.ros.org/wiki/xacro" name="my_robot">
-    <xacro:include filename="$(find gazebo_plugins)/test/multi_robot_scenario/xacro/laser/hokuyo.xacro" />
-    <xacro:include filename="$(find velodyne_description)/urdf/VLP-16.urdf.xacro" />
-    <xacro:macro name="reflect_wheel" params="suffix reflect">
-        <joint name="base_wheel_${suffix}_joint" type="continuous">
-            <origin xyz="-0.37 ${reflect*0.4} -0.99" rpy="-1.57 0.0 0.0" />
-            <axis xyz="0.0 0.0 1.0" />
-            <parent link="base" />
-            <child link="wheel_${suffix}" />
-        </joint>
-        <link name="wheel_${suffix}">
-            <origin xyz="-0.37 ${reflect*0.01} -0.99" rpy="0.0 0.0 0.0" />
-            <visual>
-                <geometry>
-                    <cylinder radius="0.2" length="0.05" />
-                </geometry>
-            </visual>
-            <collision>
-                <geometry>
-                    <cylinder radius="0.2" length="0.05" />
-                </geometry>
-            </collision>
-        </link>
-    </xacro:macro>
-    <link name="base">
-        <origin xyz="0.0 0.0 0.0" rpy="0.0 0.0 0.0" />
+<robot xmlns:xacro="http://www.ros.org/wiki/xacro" name="navvis_m6">
+    <xacro:include filename="$(find lab5_bag_package)/urdf/old_robot.xacro" />
+    <link name="base_link">
+    </link>
+    <joint name="base_link_base_joint" type="fixed">
+        <parent link="base_link" />
+        <child link="base" />
+        <origin xyz="0.07 0 1.792" rpy="0.0 ${pi} 0.0" />
+    </joint>
+    <joint name="base_link_imu_joint" type="fixed">
+        <parent link="base_link" />
+        <child link="imu" />
+        <origin xyz="0.0 0.0 0.0" rpy="3.1405788 0.0034281 3.1382064" />
+    </joint>
+    <link name="imu">
         <visual>
-            <origin xyz="0.0 0.0 -0.99" />
             <geometry>
-                <box size="0.94 0.78 0.25" />
+                <sphere radius="0.1" />
             </geometry>
         </visual>
-        <visual>
-            <origin xyz="0.23 0.0 0.0" />
-            <geometry>
-                <box size="0.10 0.78 1.9"/>
-            </geometry>
-        </visual>
-        <collision>
-            <geometry>
-                <box size="0.94 0.78 1.98" />
-            </geometry>
-        </collision>
+    <collision>
+        <geometry>
+            <sphere radius="0.1" />
+        </geometry>
+    </collision>
     </link>
-    <xacro:reflect_wheel suffix="left" reflect="1" />
-    <joint name="base_wheel_center_joint" type="continuous">
-        <origin xyz="0.57 0.0 -1.04" rpy="-1.57 0.0 0.0" />
-        <axis xyz="0.0 0.0 1.0" />
-        <parent link="base" />
-        <child link="wheel_center" />
-    </joint>
-    <link name="wheel_center">
-        <origin xyz="0.57 0.0 -1.04" rpy="0.0 0.0 0.0" />
-        <visual>
-            <geometry>
-                <cylinder radius="0.15" length="0.05" />
-            </geometry>
-        </visual>
-        <collision>
-            <geometry>
-                <cylinder radius="0.15" length="0.05" />
-            </geometry>
-        </collision>
-    </link>
-    <xacro:reflect_wheel suffix="right" reflect="-1" />
-    <xacro:VLP-16 parent="base" name="label_horiz" topic="laser_horiz/packets" hz="10" samples="440" gpu="false">
-        <origin xyz="0.2325 0.0001 0.9301" rpy="-0.0012 0.1146 -0.0015" />
-    </xacro:VLP-16>
-    <xacro:laser name="laser_vert_top_right" parent="base" xyz="0.2978 -0.1450 0.8551" rpy="-1.1760 0.6313 -1.9377" meshes="package://gazebo_plugins/test/multi_robot_scenario/meshes/laser" />
-    <xacro:laser name="laser_vert_top_left" parent="base" xyz="0.2997 0.1531 0.8543" rpy="1.1780 0.6198 1.9560" meshes="package://gazebo_plugins/test/multi_robot_scenario/meshes/laser" />
-    <xacro:laser name="laser_vert_bottom" parent="base" xyz="0.3158 -0.0021 -0.4800" rpy="3.1355 -1.3045 0.0025" meshes="package://gazebo_plugins/test/multi_robot_scenario/meshes/laser" />
 </robot>
